File: 85key.sch (KiCad schematic (older format))
At the start: 284 parts, among them IC1 ATMEGA32U4, P1 CONN_1, P2 CONN_1, P3 CONN_1, P4 CONN_1, P5 CONN_1, P6 CONN_1, SW0:0 Strg, SW0:1 Win, SW0:10 Super, SW0:11 ReStrg, SW0:12 PfeilLinks, SW0:13 PfeilRunter, SW0:14 PfeilRechts, SW0:2 Alt, SW0:6 Leer, SW0:9 AltGr, SW1:0 Shift, SW1:1 <, SW1:10 ., SW1:11 -, SW1:12 ReShift, SW1:13 PfeilHoch, SW1:14 BildRunter, SW1:2 Y, SW1:3 X, SW1:4 C, SW1:5 V, SW1:6 B, SW1:7 N, SW1:8 M, SW1:9 ,, SW2:0 Caps, SW2:1 A, SW2:10 Ö, SW2:11 Ä, SW2:12 #, SW2:13 Enter, SW2:14 BildHoch, SW2:2 S, SW2:3 D, SW2:4 F, SW2:5 G, SW2:6 H, SW2:7 J, SW2:8 K, SW2:9 L, SW3:0 Tab, SW3:1 Q, SW3:10 P, SW3:11 Ü, SW3:12 +, SW3:13 Backspace, SW3:14 Entf, SW3:2 W, SW3:3 E, SW3:4 R, SW3:5 T, SW3:6 Z, SW3:7 U, SW3:8 I, SW3:9 O, SW4:0 ^, SW4:1 1, SW4:10 0, SW4:11 ß, SW4:12 ´, SW4:13 Pause, SW4:14 Ende, SW4:2 2, SW4:3 3, SW4:4 4, SW4:5 5, SW4:6 6, SW4:7 7, SW4:8 8, SW4:9 9, SW5:0 ESC, SW5:1 F1, SW5:10 F10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

Commit message: dioden annotation korrigiert
Parts:
- gave numbers to parts that had none: 1
- renumbered D1:12 to D0:12, D1:13 to D0:13, D1:14 to D0:14
Changed lines of the file:
@@
 LIBS:valves
 LIBS:atmega32u4
-LIBS:mx1a-simple
 LIBS:85key-cache
 EELAYER 27 0
@@
 Sheet 1 1
 Title ""
-Date "18 dec 2014"
+Date "22 dec 2014"
 Rev ""
 Comp ""
@@
 $EndComp
 $Comp
-L USB_2 J?
+L USB_2 J1
 U 1 1 5492DC0C
 P 6450 7800
-F 0 "J?" H 6375 8050 60  0000 C CNN
+F 0 "J1" H 6375 8050 60  0000 C CNN
 F 1 "USB_2" H 6500 7500 60  0001 C CNN
 F 2 "" H 6450 7800 60  0000 C CNN
@@
 $EndComp
 $Comp
-L DIODE D1:12
+L DIODE D0:12
 U 1 1 5493405F
 P 12550 5650
-F 0 "D1:12" H 12550 5750 40  0000 C CNN
+F 0 "D0:12" H 12550 5750 40  0000 C CNN
 F 1 "DIODE" H 12550 5550 40  0000 C CNN
 F 2 "" H 12550 5650 60  0000 C CNN
@@
 $EndComp
 $Comp
-L DIODE D1:13
+L DIODE D0:13
 U 1 1 549340BA
 P 13450 5650
-F 0 "D1:13" H 13450 5750 40  0000 C CNN
+F 0 "D0:13" H 13450 5750 40  0000 C CNN
 F 1 "DIODE" H 13450 5550 40  0000 C CNN
 F 2 "" H 13450 5650 60  0000 C CNN
@@
 $EndComp
 $Comp
-L DIODE D1:14
+L DIODE D0:14
 U 1 1 54934137
 P 14350 5650
-F 0 "D1:14" H 14350 5750 40  0000 C CNN
+F 0 "D0:14" H 14350 5750 40  0000 C CNN
 F 1 "DIODE" H 14350 5550 40  0000 C CNN
 F 2 "" H 14350 5650 60  0000 C CNN
